Commit message: 摄像头朝向正确，但是点云方向错误

File: urdf/my_gen3_with_camera.urdf.xacro (robot description, xacro)
@@ -6,5 +6,6 @@
   <xacro:arg name="sim" default="true"/>
   <xacro:arg name="prefix" default=""/>
-  <xacro:arg name="gripper" default="robotiq_2f_85"/> <xacro:arg name="robot_name" default="my_gen3"/>
+  <xacro:arg name="gripper" default="robotiq_2f_85"/>
+  <xacro:arg name="robot_name" default="my_gen3"/>
   <xacro:property name="arm" value="$(arg arm)"/>
   <xacro:property name="dof" value="$(arg dof)"/>
@@ -28,12 +29,6 @@
                    prefix="${prefix}" />
   </xacro:unless>
-  <link name="${prefix}camera_link_sim"/>
-  <joint name="${prefix}camera_mount_joint" type="fixed">
-    <parent link="${prefix}tool_frame"/>
-    <child link="${prefix}camera_link_sim"/>
-    <origin xyz="0.0 0.0 0.0" rpy="0.0 0.0 0.0"/>
-  </joint>
   <xacro:if value="${sim}">
-    <gazebo reference="${prefix}camera_link_sim">
+    <gazebo reference="${prefix}camera_depth_frame">
       <sensor type="depth" name="realsense_sim">
         <always_on>true</always_on>
@@ -47,6 +42,6 @@
           </image>
           <clip>
-            <near>0.1</near>
-            <far>100</far>
+            <near>0.2</near>
+            <far>8.0</far>
           </clip>
         </camera>
@@ -54,8 +49,10 @@
           <baseline>0.2</baseline>
           <pointCloudCutoff>0.1</pointCloudCutoff>
-          <pointCloudCutoffMax>5.0</pointCloudCutoffMax>
+          <alwaysOn>true</alwaysOn>
           <robotNamespace>${robot_name}</robotNamespace>
           <cameraName>camera</cameraName>
-          <frameName>${prefix}camera_link_sim</frameName>
+          <updateRate>10</updateRate>
+          <frameName>camera_depth</frameName>
+          <pointCloudCutoff>0.4</pointCloudCutoff>
           <imageTopicName>color/image_raw</imageTopicName>
           <depthImageTopicName>depth/image_raw</depthImageTopicName>
